File: Frekeys.kicad_sch (KiCad schematic)
At the start: 12 parts, among them J1 AudioPlug3, SW1 RotaryEncoder_Switch, U1 CR2013-MI2120, U2 ESP32-S3-DevKitC, U3 74HC165, U4 74HC165

Commit message: Making.. 2
Parts:
- added R10, R5, R6, R7, R8, R9: 10k, Resistor_SMD:R_0805_2012Metric, symbol Device:R
Connections:
- net Keyboard/R3: now also R6.2; no longer U4.3 (D4)
- net Keyboard/R4: now also R7.2; no longer U4.14 (D3)
- net Keyboard/R5: now also R8.2; no longer U4.13 (D2)
- net Keyboard/R6: now also R10.2; no longer U4.12 (D1)
- net Keyboard/R7: now also R5.2; no longer U4.11 (D0)
- new net: R5.1, U4.11 (D0)
- new net: R8.1, U4.13 (D2)
- new net: R7.1, U4.14 (D3)
- new net: R10.1, U4.12 (D1)
- new net: R6.1, U4.3 (D4)

Commit message: making.... 3
making.... 3
Parts:
- added R11, R12, R13, R14, R15, R16, R17, R18, R19, R20: 10k, Resistor_SMD:R_0805_2012Metric, symbol Device:R
Connections:
- net Keyboard/C: now also R16.2; no longer U3.6 (D7)
- net Keyboard/C1: now also R15.2; no longer U3.5 (D6)
- net Keyboard/C2: now also R14.2; no longer U3.4 (D5)
- net Keyboard/C3: now also R17.2; no longer U3.3 (D4)
- net Keyboard/C4: now also R18.2; no longer U3.14 (D3)
- net Keyboard/C5: now also R19.2; no longer U3.13 (D2)
- net Keyboard/C6: now also R20.2; no longer U3.12 (D1)
- net Keyboard/C7: now also R12.2; no longer U3.11 (D0)
- net Keyboard/R: now also R11.2; no longer U4.6 (D7)
- net Keyboard/R1: now also R9.2; no longer U4.5 (D6)
- net Keyboard/R2: now also R13.2; no longer U4.4 (D5)
- net at R9.1: now also U4.5 (D6)
- new net: R15.1, U3.5 (D6)
- new net: R13.1, U4.4 (D5)
- new net: R14.1, U3.4 (D5)
- new net: R16.1, U3.6 (D7)
- new net: R12.1, U3.11 (D0)
- new net: R20.1, U3.12 (D1)
- new net: R19.1, U3.13 (D2)
- new net: R18.1, U3.14 (D3)
- new net: R17.1, U3.3 (D4)
- new net: R11.1, U4.6 (D7)
Other:
- moved on the sheet: R10, R5, R7, R8, R9

Commit message: Maybe Final
Parts:
- U3, U4: footprint Package_DIP:DIP-16_W7.62mm -> Package_SO:SOIC-16_3.9x9.9mm_P1.27mm
Changed lines of the file:
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@@
 			)
 		)
-		(property "Footprint" "Package_DIP:DIP-16_W7.62mm"
+		(property "Footprint" "Package_SO:SOIC-16_3.9x9.9mm_P1.27mm"
 			(at 215.9 81.28 0)
 			(effects
@@
 			)
 		)
-		(property "Footprint" "Package_DIP:DIP-16_W7.62mm"
+		(property "Footprint" "Package_SO:SOIC-16_3.9x9.9mm_P1.27mm"
 			(at 254 82.55 0)
 			(effects
