File: Frekeys.kicad_pcb (KiCad board)
At the start: 2 copper layers, 1.4 x 13 mm, 140 parts, among them J1 AudioPlug3, SW1 RotaryEncoder_Switch, SW10 SW_Push, SW11 SW_Push, SW12 SW_Push, SW13 SW_Push, SW14 SW_Push, SW15 SW_Push, SW16 SW_Push, SW17 SW_Push, SW18 SW_Push, SW19 SW_Push, SW2 SW_Push, SW20 SW_Push, SW21 SW_Push, SW22 SW_Push, SW23 SW_Push, SW24 SW_Push, SW25 SW_Push, SW26 SW_Push, SW27 SW_Push, SW28 SW_Push, SW29 SW_Push, SW3 SW_Push, SW30 SW_Push, SW31 SW_Push, SW32 SW_Push, SW33 SW_Push, SW34 SW_Push, SW35 SW_Push, SW36 SW_Push, SW37 SW_Push, SW38 SW_Push, SW39 SW_Push, SW4 SW_Push, SW40 SW_Push, SW41 SW_Push, SW42 SW_Push, SW43 SW_Push, SW44 SW_Push, SW45 SW_Push, SW46 SW_Push, SW47 SW_Push, SW48 SW_Push, SW49 SW_Push, SW5 SW_Push, SW50 SW_Push, SW51 SW_Push, SW52 SW_Push, SW53 SW_Push, SW54 SW_Push, SW55 SW_Push, SW56 SW_Push, SW57 SW_Push, SW58 SW_Push, SW59 SW_Push, SW6 SW_Push, SW60 SW_Push, SW61 SW_Push, SW62 SW_Push, SW63 SW_Push, SW64 SW_Push, SW65 SW_Push, SW7 SW_Push, SW8 SW_Push, SW9 SW_Push, U1 CR2013-MI2120, U2 ESP32-S3-DevKitC, U3 74HC165, U4 74HC165

Commit message: Update Frekeys.kicad_pcb
Nope comment
Parts:
- added R10: 10k, Resistor_SMD:R_0805_2012Metric, F.Cu at (230.4, 84.6)
- added R11: 10k, Resistor_SMD:R_0805_2012Metric, F.Cu at (233.4, 99.9)
- added R12: 10k, Resistor_SMD:R_0805_2012Metric, F.Cu at (233.0, 104.4)
- added R13: 10k, Resistor_SMD:R_0805_2012Metric, F.Cu at (228.0, 100.0)
- added R14: 10k, Resistor_SMD:R_0805_2012Metric, F.Cu at (227.5, 120.5)
- added R15: 10k, Resistor_SMD:R_0805_2012Metric, F.Cu at (230.0, 120.5)
- added R16: 10k, Resistor_SMD:R_0805_2012Metric, F.Cu at (233.0, 120.5)
- added R17: 10k, Resistor_SMD:R_0805_2012Metric, F.Cu at (225.0, 120.5)
- added R18: 10k, Resistor_SMD:R_0805_2012Metric, F.Cu at (224.5, 104.5)
- added R19: 10k, Resistor_SMD:R_0805_2012Metric, F.Cu at (226.5, 104.5)
- added R20: 10k, Resistor_SMD:R_0805_2012Metric, F.Cu at (230.0, 104.6)
- added R5: 10k, Resistor_SMD:R_0805_2012Metric, F.Cu at (233.1, 84.6)
- added R6: 10k, Resistor_SMD:R_0805_2012Metric, F.Cu at (225.0, 100.0)
- added R7: 10k, Resistor_SMD:R_0805_2012Metric, F.Cu at (224.5, 84.6)
- added R8: 10k, Resistor_SMD:R_0805_2012Metric, F.Cu at (227.4, 84.6)
- added R9: 10k, Resistor_SMD:R_0805_2012Metric, F.Cu at (230.5, 99.9)
- moved D1 110.6 mm to (35.1, 15.5)
- moved D2 73.5 mm to (35.1, 32.0)
- moved D3 60.6 mm to (35.1, 48.0)
- moved D4 48.8 mm to (35.1, 63.0)
- moved D5 36.3 mm to (35.0, 78.6)
- moved D6 23.7 mm to (35.0, 94.5)
- moved D7 12.2 mm to (34.9, 110.0)
- moved U3 5.80 mm to (220.1, 116.8)
- moved D8 0.50 mm to (35.1, 125.5)
Connections:
- U3 pad 11: /Keyboard/C7 -> Net-(U3-D0)
- U3 pad 12: /Keyboard/C6 -> Net-(U3-D1)
- U3 pad 13: /Keyboard/C5 -> Net-(U3-D2)
- U3 pad 14: /Keyboard/C4 -> Net-(U3-D3)
- U3 pad 3: /Keyboard/C3 -> Net-(U3-D4)
- U3 pad 4: /Keyboard/C2 -> Net-(U3-D5)
- U3 pad 5: /Keyboard/C1 -> Net-(U3-D6)
- U3 pad 6: /Keyboard/C -> Net-(U3-D7)
- U4 pad 11: /Keyboard/R7 -> Net-(U4-D0)
- U4 pad 12: /Keyboard/R6 -> Net-(U4-D1)
- U4 pad 13: /Keyboard/R5 -> Net-(U4-D2)
- U4 pad 14: /Keyboard/R4 -> Net-(U4-D3)
- U4 pad 3: /Keyboard/R3 -> Net-(U4-D4)
- U4 pad 4: /Keyboard/R2 -> Net-(U4-D5)
- U4 pad 5: /Keyboard/R1 -> Net-(U4-D6)
- U4 pad 6: /Keyboard/R -> Net-(U4-D7)

Commit message: a
a
Parts:
- moved D9 144.4 mm to (54.6, 20.6), turned to 90 degrees
- moved D17 137.9 mm to (77.5, 20.5), turned to 90 degrees
- moved D10 128.1 mm to (54.5, 39.9), turned to 90 degrees
- moved D18 121.8 mm to (77.5, 40.0), turned to 90 degrees
- moved D11 111.7 mm to (54.5, 59.4), turned to 90 degrees
- moved D19 105.8 mm to (77.5, 59.5), turned to 90 degrees
- moved D20 90.1 mm to (77.5, 78.9), turned to 90 degrees
- moved D34 79.1 mm to (95.0, 196.6)
- moved D45 79.1 mm to (99.4, 196.6)
- moved D56 79.1 mm to (103.9, 196.6)
- moved D21 74.6 mm to (77.5, 98.5), turned to 90 degrees
- moved D46 67.6 mm to (99.5, 200.3)
- moved D49 67.6 mm to (99.5, 209.5)
- moved D52 67.6 mm to (99.5, 218.6)
- moved D53 67.6 mm to (99.5, 221.6)
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
Commit message: ダイオードの場所設定OK
Parts:
- moved D33 209.6 mm to (121.5, 20.4), turned to 90 degrees
- moved D41 204.2 mm to (144.5, 20.4), turned to 90 degrees
- moved D57 203.2 mm to (198.5, 20.4), turned to 90 degrees
- moved D49 202.3 mm to (173.0, 20.9), turned to 90 degrees
- moved D58 188.3 mm to (198.5, 40.5), turned to 90 degrees
- moved D42 188.3 mm to (144.5, 39.9), turned to 90 degrees
- moved D50 187.1 mm to (173.0, 40.4), turned to 90 degrees
- moved D25 183.2 mm to (100.0, 20.4), turned to 90 degrees
- moved D59 174.8 mm to (198.5, 59.4), turned to 90 degrees
- moved D43 172.4 mm to (144.5, 59.5), turned to 90 degrees
- moved D51 172.1 mm to (173.0, 59.9), turned to 90 degrees
- moved D26 166.7 mm to (100.0, 40.0), turned to 90 degrees
- moved D60 161.2 mm to (198.5, 78.9), turned to 90 degrees
- moved D34 158.8 mm to (121.5, 40.0), turned to 90 degrees
- moved D52 157.4 mm to (173.0, 79.4), turned to 90 degrees
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
Commit message: 形状ほぼ完成
Parts:
- SW14, SW22, SW6: footprint PCM_Switch_Keyboard_Hotswap_Kailh:SW_Hotswap_Kailh_MX_1.00u -> PCM_Switch_Keyboard_Hotswap_Kailh:SW_Hotswap_Kailh_MX_1.25u
- SW3: footprint PCM_Switch_Keyboard_Hotswap_Kailh:SW_Hotswap_Kailh_MX_1.00u -> PCM_Switch_Keyboard_Hotswap_Kailh:SW_Hotswap_Kailh_MX_1.50u
- SW38: footprint PCM_Switch_Keyboard_Hotswap_Kailh:SW_Hotswap_Kailh_MX_1.00u -> PCM_Switch_Keyboard_Hotswap_Kailh:SW_Hotswap_Kailh_MX_Plated_6.00u
- SW4: footprint PCM_Switch_Keyboard_Hotswap_Kailh:SW_Hotswap_Kailh_MX_1.00u -> PCM_Switch_Keyboard_Hotswap_Kailh:SW_Hotswap_Kailh_MX_1.75u
- SW5, SW63: footprint PCM_Switch_Keyboard_Hotswap_Kailh:SW_Hotswap_Kailh_MX_1.00u -> PCM_Switch_Keyboard_Hotswap_Kailh:SW_Hotswap_Kailh_MX_2.00u
- SW64: footprint PCM_Switch_Keyboard_Hotswap_Kailh:SW_Hotswap_Kailh_MX_1.00u -> PCM_Switch_Keyboard_Hotswap_Kailh:SW_Hotswap_Kailh_MX_ISOEnter
- moved D8 248.6 mm to (261.2, 59.4)
- moved SW9 248.6 mm to (252.6, 60.5)
- moved D16 225.5 mm to (266.1, 79.0)
- moved SW17 225.5 mm to (257.6, 80.0)
- moved D7 223.2 mm to (241.6, 59.4)
- moved SW8 223.2 mm to (233.0, 60.5)
- moved D24 222.2 mm to (285.6, 78.9)
- moved SW25 222.2 mm to (277.1, 80.0)
- moved D15 200.8 mm to (246.6, 79.0)
- moved SW16 200.8 mm to (238.1, 80.0)
- moved D6 179.3 mm to (207.6, 78.9)
- moved SW7 179.3 mm to (198.9, 80.0)
- moved SW24 160.5 mm to (218.5, 80.0)
- moved D23 160.5 mm to (227.0, 79.0)
- moved SW15 159.1 mm to (194.0, 60.5)
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
Commit message: Maybe Final
Parts:
- SW38: footprint PCM_Switch_Keyboard_Hotswap_Kailh:SW_Hotswap_Kailh_MX_Plated_6.00u -> PCM_Switch_Keyboard_Hotswap_Kailh:SW_Hotswap_Kailh_MX_6.00u
- U3, U4: footprint Package_DIP:DIP-16_W7.62mm -> Package_SO:SOIC-16_3.9x9.9mm_P1.27mm
- moved D64 147.6 mm to (329.0, 33.4)
- moved SW65 147.6 mm to (320.5, 34.0)
- moved D32 128.6 mm to (328.9, 111.5)
- moved SW33 128.6 mm to (320.5, 112.5)
- moved D56 127.0 mm to (328.9, 52.5)
- moved SW57 127.0 mm to (320.5, 53.5)
- moved D48 111.7 mm to (328.9, 72.0)
- moved SW49 111.7 mm to (320.4, 73.0)
- moved D40 103.1 mm to (329.0, 92.0)
- moved SW41 103.1 mm to (320.5, 93.0)
- moved R11 38.5 mm to (336.3, 64.6)
- moved R20 38.5 mm to (338.8, 51.6)
- moved R9 38.5 mm to (339.3, 64.6)
- moved R10 38.5 mm to (339.4, 79.9)
- moved R12 38.5 mm to (335.8, 51.8)
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Other:
- board size 1.4 x 13 mm -> 403 x 108 mm

Commit message: maybe final
maybe final
Parts:
- added REF**: Stabilizer_Cherry_MX_6.25u, PCM_Mounting_Keyboard_Stabilizer:Stabilizer_Cherry_MX_6.25u, F.Cu at (178.7, 111.7)
- added REF**: Stabilizer_Cherry_MX_2.00u, PCM_Mounting_Keyboard_Stabilizer:Stabilizer_Cherry_MX_2.00u, F.Cu at (44.4, 93.0)
- added REF**: Stabilizer_Cherry_MX_2.00u, PCM_Mounting_Keyboard_Stabilizer:Stabilizer_Cherry_MX_2.00u, F.Cu at (284.1, 63.5)
- added REF**: Stabilizer_Cherry_MX_2.00u, PCM_Mounting_Keyboard_Stabilizer:Stabilizer_Cherry_MX_2.00u, F.Cu at (278.4, 33.6)
- D1, D10, D11, D12, D13, D14, D15, D16, D17, D18, D19, D2, D20, D21, D22, D23, D24, D25, D26, D27, D28, D29, D3, D30, D31, D32, D33, D34, D35, D36, D37, D38, D39, D4, D40, D41, D42, D43, D44, D45, D46, D47, D48, D49, D5, D50, D51, D52, D53, D54, D55, D56, D57, D58, D59, D6, D60, D61, D62, D63, D64, D7, D8, D9, R10, R11, R12, R13, R14, R15, R16, R17, R18, R19, R20, R5, R6, R7, R8, R9, U3, U4: moved to B.Cu
- SW38: footprint PCM_Switch_Keyboard_Hotswap_Kailh:SW_Hotswap_Kailh_MX_6.00u -> PCM_Switch_Keyboard_Hotswap_Kailh:SW_Hotswap_Kailh_MX_6.25u
- moved R7 9.56 mm to (335.7, 79.9)
- moved R12 9.44 mm to (345.2, 51.8)
- moved R6 8.56 mm to (336.2, 64.5)
- moved R16 8.44 mm to (344.7, 36.7)
- moved R11 8.34 mm to (344.6, 64.6)
- moved R17 7.56 mm to (336.7, 36.7)
- moved R18 7.56 mm to (336.7, 51.7)
- moved R5 7.54 mm to (344.2, 79.9)
- moved R8 3.66 mm to (338.6, 79.9)
- moved R19 3.56 mm to (338.7, 51.7)
- moved R20 3.44 mm to (342.2, 51.6)
- moved D37 2.98 mm to (189.9, 107.5), turned to 0 degrees
- moved R13 2.56 mm to (339.2, 64.5)
- moved R14 2.56 mm to (339.2, 36.7)
- moved R15 2.44 mm to (341.7, 36.7)
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Routing:
- net /Keyboard/C3: track 0.00 -> 486.2 mm, vias 0 -> 22
- net /Keyboard/C: track 0.00 -> 442.6 mm, vias 0 -> 4
- net /Keyboard/C1: track 0.00 -> 441.6 mm, vias 0 -> 11
- net /Keyboard/C2: track 0.00 -> 440.7 mm, vias 0 -> 15
- net /Keyboard/C6: track 0.00 -> 402.9 mm, vias 0 -> 17
- net /Keyboard/C4: track 0.00 -> 395.8 mm, vias 0 -> 14
- net /Keyboard/C5: track 0.00 -> 385.2 mm, vias 0 -> 12
- net /Keyboard/R: track 0.00 -> 370.7 mm, vias 0 -> 2
- net /Keyboard/R2: track 0.00 -> 359.3 mm, vias 0 -> 6
- net /Keyboard/C7: track 0.00 -> 351.0 mm, vias 0 -> 11
- net /Keyboard/R3: track 0.00 -> 331.2 mm, vias 0 -> 12
- net /Keyboard/R4: track 0.00 -> 323.7 mm, vias 0 -> 2
- net /Keyboard/R1: track 0.00 -> 318.9 mm, vias 0 -> 6
- net /Keyboard/R5: track 0.00 -> 239.7 mm, vias 0 -> 2
- net GND: track 0.00 -> 226.1 mm, vias 0 -> 1
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- added copper zone on F.Cu, net GND

Commit message: Final Commit
Parts:
- C1, C2, R1, R2, R3, R4: moved to B.Cu
- moved R4 5.53 mm to (391.4, 96.0)
- moved R3 1.55 mm to (383.6, 100.5)
- moved R2 0.57 mm to (388.0, 99.5)
Routing:
- net Net-(U2-GPIO17/ADC2_CH6): track 108.3 -> 63.1 mm, vias 1 -> 0
- net Net-(U1-VCC): track 113.7 -> 123.3 mm, vias 3 -> 7
- net Net-(U2-GPIO48): track 104.6 -> 97.5 mm
- net Net-(U2-GPIO46): track 72.7 -> 74.8 mm, vias 0 -> 1
- net Net-(U2-GPIO47): track 86.4 -> 88.1 mm, vias 0 -> 1
- net Net-(U2-GPIO18/ADC2_CH7): track 56.5 -> 54.8 mm, vias 1 -> 0
- net Net-(U1-SD_SCK): track 76.2 -> 77.4 mm, vias 3 -> 2
- net Net-(U2-CHIP_PU): vias 0 -> 1
- net /Keyboard/C1: vias 11 -> 10
Other:
- outline, holes or cut-outs redrawn
